File: UccMicroDuino/UccMicroDuino.kicad_pcb (KiCad board)
At the start: 2 copper layers, 8 parts, among them J1 Conn_01x10_Socket, J2 USB_A, U1 ATtiny85-20S

Commit message: Add files via upload
Parts:
- added D4: LED Green, ledSmd:ledSMD, F.Cu at (225.8, 91.0)
- added D5: LED Red, ledSmd:ledSMD, F.Cu at (207.0, 91.0)
- added R2: 68Ω 5% 1/8W, Resistor_SMD:R_0805_2012Metric_Pad1.20x1.40mm_HandSolder, F.Cu at (210.7, 73.0)
- added R3: 68Ω 5% 1/8W, Resistor_SMD:R_0805_2012Metric_Pad1.20x1.40mm_HandSolder, F.Cu at (223.0, 73.0)
- added R4: 68Ω 5% 1/8W, Resistor_SMD:R_0805_2012Metric_Pad1.20x1.40mm_HandSolder, F.Cu at (215.0, 84.0)
- added R5: 330Ω 5% 1/8w, Resistor_SMD:R_0805_2012Metric_Pad1.20x1.40mm_HandSolder, F.Cu at (206.0, 96.0)
- C1: value C -> 0.1u
- D2: value D_Zener -> 3.6V 1/2mw
- D3: value LED -> 3.6V 1/2mw; footprint ledSmd:ledSMD -> Diode_SMD:D_SOD-123
- J1: value Conn_01x10_Socket -> Pcb USB type A; footprint Connector_PinHeader_2.54mm:PinHeader_1x10_P2.54mm_Vertical -> embeddedPcbUsb:USB_A_UCC
- J2: value USB_A -> Conn_01x10_Socket; footprint embeddedPcbUsb:USB_A_UCC -> Connector_PinHeader_2.54mm:PinHeader_1x10_P2.54mm_Vertical
- R1: value R -> 1/5KΩ 5% 1/8W
- U1: footprint Package_SO:SOIC-8W_5.3x5.3mm_P1.27mm -> Package_SO:SOIC-8_5.3x5.3mm_P1.27mm
- moved U1 99.3 mm to (231.0, 81.0), turned to 180 degrees
- moved D3 88.9 mm to (222.7, 69.0)
- moved J2 88.0 mm to (217.0, 95.0), turned to 90 degrees
- moved J1 84.4 mm to (208.2, 61.0), turned to -90 degrees
- moved D2 83.5 mm to (210.0, 69.0)
- moved D1 76.7 mm to (206.0, 80.0)
- moved C1 69.5 mm to (206.0, 84.0)
- moved R1 67.6 mm to (206.0, 75.0)
Connections:
- C1 pad 1: unconnected-(C1-Pad1) -> +5V
- C1 pad 2: unconnected-(C1-Pad2) -> GND
- D1 pad 2: unconnected-(D1-A-Pad2) -> Net-(D1-A)
- D2 pad 1: unconnected-(D2-K-Pad1) -> Net-(D2-K)
- D2 pad 2: unconnected-(D2-A-Pad2) -> GND
- D3 pad 1: unconnected-(D3-K-Pad1) -> Net-(D3-K)
- D3 pad 2: unconnected-(D3-A-Pad2) -> GND
- J1 pad 1: unconnected-(J1-Pin_1-Pad1) -> Net-(D1-A)
- J1 pad 2: unconnected-(J1-Pin_2-Pad2) -> Net-(D2-K)
- J1 pad 3: unconnected-(J1-Pin_3-Pad3) -> Net-(D3-K)
- J1 pad 4: unconnected-(J1-Pin_4-Pad4) -> GND
- J2 pad 1: unconnected-(J2-VBUS-Pad1) -> +5V
- J2 pad 2: unconnected-(J2-D--Pad2) -> GND
- J2 pad 4: unconnected-(J2-GND-Pad4) -> Net-(J2-Pin_4)
- R1 pad 2: unconnected-(R1-Pad2) -> Net-(D2-K)
- U1 pad 1: unconnected-(U1-~{RESET}/PB5-Pad1) -> Net-(J2-Pin_9)
- U1 pad 2: unconnected-(U1-XTAL1/PB3-Pad2) -> Net-(J2-Pin_7)
- U1 pad 3: unconnected-(U1-XTAL2/PB4-Pad3) -> Net-(J2-Pin_8)
- U1 pad 4: unconnected-(U1-GND-Pad4) -> GND
- U1 pad 5: unconnected-(U1-AREF/PB0-Pad5) -> Net-(J2-Pin_4)
- U1 pad 6: unconnected-(U1-PB1-Pad6) -> Net-(D4-A)
- U1 pad 7: unconnected-(U1-PB2-Pad7) -> Net-(J2-Pin_6)
- U1 pad 8: unconnected-(U1-VCC-Pad8) -> +5V
Routing:
- net GND: track 0.00 -> 125.8 mm
- net Net-(J2-Pin_7): track 0.00 -> 66.6 mm
- net +5V: track 0.00 -> 63.6 mm
- net Net-(J2-Pin_8): track 0.00 -> 30.2 mm
- net Net-(D1-A): track 0.00 -> 26.4 mm
- net Net-(D3-K): track 0.00 -> 24.5 mm
- net Net-(J2-Pin_4): track 0.00 -> 19.0 mm
- net Net-(D4-A): track 0.00 -> 17.4 mm
- net Net-(D2-K): track 0.00 -> 16.2 mm
- net Net-(J2-Pin_6): track 0.00 -> 15.9 mm
- net (no net): track 0.00 -> 14.0 mm
- net Net-(J2-Pin_9): track 0.00 -> 13.5 mm
- net Net-(D4-K): track 0.00 -> 10.9 mm
- net Net-(D5-K): track 0.00 -> 5.08 mm
Other:
- board outline added: 45 x 44 mm
